File: _autosave-CatEars.kicad_pcb (KiCad board)
At the start: 2 copper layers, 65.1 x 39 mm, 52 parts, among them U2 AP2112K-3.3

Commit message: Minor board design revision to allow more space to connect battery and easier assembly
Parts:
- removed 3V3, GND: Conn_01x01, TestPoint:TestPoint_Pad_D1.0mm
- removed the REF** at (232.4, 135.6)
- removed the REF** at (229.9, 132.9)
- removed the REF** at (232.0, 134.8)
- removed the REF** at (231.6, 134.0)
- removed the REF** at (231.2, 133.2)
- removed the REF** at (230.8, 132.3)
- removed the REF** at (231.4, 136.2)
- removed the REF** at (231.0, 135.4)
- removed the REF** at (230.6, 134.6)
- removed the REF** at (230.3, 133.7)
- added REF**: 1mm_npth, footprints:1mm_npth, F.Cu at (231.5, 135.0)
- added REF**: 1mm_npth, footprints:1mm_npth, F.Cu at (230.8, 133.4)
- added Reset: SW_Push, Button_Switch_SMD:SW_SPST_EVQPE1, F.Cu at (218.7, 144.5)
- C8: moved to B.Cu
- Microcontroller :D: renamed from ATSAMD21E18
- NekoMimiLink: renamed from NML Input
- moved J31 13.1 mm to (207.8, 140.7)
- moved NekoMimiLink 8.85 mm to (216.3, 149.4), turned to 90 degrees
- moved D8 8.35 mm to (208.3, 141.2), turned to 90 degrees
- moved J32 8.29 mm to (210.8, 140.7)
- moved R1 7.99 mm to (216.7, 139.7)
- moved U2 7.45 mm to (212.3, 143.8)
- moved C6 6.87 mm to (220.0, 139.7), turned to 270 degrees
- moved D7 5.15 mm to (228.1, 142.2), turned to 180 degrees
- moved Microcontroller :D 4.59 mm to (218.8, 140.6)
- moved C8 3.57 mm to (227.1, 138.7), turned to 90 degrees
- moved R6 2.41 mm to (218.9, 131.6)
- moved D6 1.78 mm to (218.9, 128.8)
- moved C1 1.20 mm to (210.6, 147.8)
- moved C5 1.14 mm to (226.8, 147.8)
- moved Battery! 0.66 mm to (208.0, 147.7)
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- renumbered BT1 to Battery!, 31 to J31, 32 to J32, D0 to Power!
Routing:
- net Net-(C21-Pad2): track 38.1 -> 158.5 mm, vias 3 -> 7
- net +3V3: track 101.8 -> 140.5 mm, vias 6 -> 10
- net GND: track 110.2 -> 138.5 mm, vias 12 -> 8
- net Net-(D1-Pad4): track 3.37 -> 19.5 mm
- net Net-(R1-Pad1): track 18.5 -> 4.11 mm
- net Net-(J31-Pad1): track 4.48 -> 14.1 mm
- net Net-(C21-Pad1): track 72.1 -> 80.1 mm, vias 1 -> 0
- net VBUS: track 12.3 -> 5.36 mm
- net Net-(C8-Pad1): track 19.4 -> 24.9 mm, vias 0 -> 1
- net Net-(D5-Pad2): track 6.67 -> 11.3 mm
- net +BATT: track 11.6 -> 7.34 mm
- net Net-(H1-Pad1): track 22.8 -> 26.9 mm
- net /USB_D-: track 15.3 -> 11.7 mm
- net Net-(SW1-Pad1): track 0.00 -> 3.56 mm, vias 0 -> 1
- net Net-(C6-Pad2): track 8.65 -> 5.27 mm
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Other:
- board text added: "Meow Meow Ears v3 by @GalaxyAllieCat 2020-02-06"
- board text removed: "+"
- board text removed: "-"
- board text removed: "Meow Meow Ears v3b by @GalaxyAllieCat 2020-03-01"
